File: saturnine_bottom-left.kicad_pcb (KiCad board)
At the start: 2 copper layers, 182.3 x 181.8 mm, 4 parts

Commit message: commit correct files
Parts:
- removed ** (x3): Val**, kbd:1pin_conn
- removed Jack0: TRRS, Kailh:TRRS-PJ-DPB2
Routing:
- net (no net): track 96.8 -> 0.00 mm
Other:
- board size 182.3 x 181.8 mm -> 99 x 80.1 mm
